Commit message: doubled ratios for defining cylinder and triangular shapes

File: urdf/blue_cylinder.urdf (robot description, URDF)
Before this commit: robot blue_cylinder, 1 links, 0 joints
Links:
- link base_link: geometry collision cylinder length=0.025 radius=0.065; visual cylinder length=0.025 radius=0.065

File: urdf/red_cylinder.urdf (robot description, URDF)
Before this commit: robot red_cylinder, 1 links, 0 joints
Links:
- link base_link: geometry collision cylinder length=0.025 radius=0.065; visual cylinder length=0.025 radius=0.065

File: urdf/yellow_cylinder.urdf (robot description, URDF)
Before this commit: robot yellow_cylinder, 1 links, 0 joints
Links:
- link base_link: geometry collision cylinder length=0.025 radius=0.065; visual cylinder length=0.025 radius=0.065

Commit message: changed mass values of cylinders

File: urdf/blue_cylinder.urdf (robot description, URDF)
Before this commit: robot blue_cylinder, 1 links, 0 joints
Links:
- link base_link: mass 0.00001 -> 0.1

File: urdf/red_cylinder.urdf (robot description, URDF)
Before this commit: robot red_cylinder, 1 links, 0 joints
Links:
- link base_link: mass 0.00001 -> 0.1

File: urdf/yellow_cylinder.urdf (robot description, URDF)
Before this commit: robot yellow_cylinder, 1 links, 0 joints
Links:
- link base_link: mass 0.00001 -> 0.1
