Commit message: fixed triangle urdf files; gripper now picks them up properly

File: urdf/blue_triangle.urdf (robot description, URDF)
Before this commit: robot red_triangle, 1 links, 0 joints
Links:
- link base_link: mass 0.00005 -> 0.01

File: urdf/red_triangle.urdf (robot description, URDF)
Before this commit: robot red_triangle, 1 links, 0 joints
Links:
- link base_link: mass 0.000005 -> 0.01

File: urdf/yellow_triangle.urdf (robot description, URDF)
Before this commit: robot red_triangle, 1 links, 0 joints
Links:
- link base_link: mass 0.000005 -> 0.01
