Commit message: urdf: updated urdf files to have similar sizes

File: urdf/blue_box.urdf (robot description, URDF)
Before this commit: robot blue_box, 1 links, 0 joints
Links:
- link base_link: geometry collision box size=0.075 0.075 0.025; visual box size=0.075 0.075 0.025

File: urdf/blue_cylinder.urdf (robot description, URDF)
Before this commit: robot blue_cylinder, 1 links, 0 joints
Links:
- link base_link: geometry collision cylinder length=0.025 radius=0.0325; visual cylinder length=0.025 radius=0.0325

File: urdf/red_box.urdf (robot description, URDF)
Before this commit: robot red_box, 1 links, 0 joints
Links:
- link base_link: geometry collision box size=0.075 0.075 0.025; visual box size=0.075 0.075 0.025

File: urdf/red_cylinder.urdf (robot description, URDF)
Before this commit: robot red_cylinder, 1 links, 0 joints
Links:
- link base_link: geometry collision cylinder length=0.025 radius=0.0325; visual cylinder length=0.025 radius=0.0325

File: urdf/yellow_box.urdf (robot description, URDF)
Before this commit: robot yellow_box, 1 links, 0 joints
Links:
- link base_link: geometry collision box size=0.075 0.075 0.025; visual box size=0.075 0.075 0.025

File: urdf/yellow_cylinder.urdf (robot description, URDF)
Before this commit: robot yellow_cylinder, 1 links, 0 joints
Links:
- link base_link: geometry collision cylinder length=0.025 radius=0.0325; visual cylinder length=0.025 radius=0.0325

Commit message: changes to urdf files to increase size/friction and decrease mass

File: urdf/blue_box.urdf (robot description, URDF)
Before this commit: robot blue_box, 1 links, 0 joints
Links:
- link base_link: mass 0.05 -> 0.005; geometry collision box size=0.125 0.125 0.025; visual box size=0.125 0.125 0.025

File: urdf/blue_cylinder.urdf (robot description, URDF)
Before this commit: robot blue_cylinder, 1 links, 0 joints
Links:
- link base_link: mass 0.1 -> 0.01

File: urdf/blue_triangle.urdf (robot description, URDF)
Before this commit: robot red_triangle, 1 links, 0 joints
Links:
- link base_link: mass 0.05 -> 0.00005

File: urdf/red_box.urdf (robot description, URDF)
Before this commit: robot red_box, 1 links, 0 joints
Links:
- link base_link: mass 0.05 -> 0.005; geometry collision box size=0.125 0.125 0.025; visual box size=0.125 0.125 0.025

File: urdf/red_cylinder.urdf (robot description, URDF)
Before this commit: robot red_cylinder, 1 links, 0 joints
Links:
- link base_link: mass 0.1 -> 0.005

File: urdf/red_triangle.urdf (robot description, URDF)
Before this commit: robot red_triangle, 1 links, 0 joints
Links:
- link base_link: mass 0.05 -> 0.000005

File: urdf/yellow_box.urdf (robot description, URDF)
Before this commit: robot yellow_box, 1 links, 0 joints
Links:
- link base_link: mass 0.05 -> 0.000005; geometry collision box size=0.125 0.125 0.025; visual box size=0.125 0.125 0.025

File: urdf/yellow_cylinder.urdf (robot description, URDF)
Before this commit: robot yellow_cylinder, 1 links, 0 joints
Links:
- link base_link: mass 0.1 -> 0.005

File: urdf/yellow_triangle.urdf (robot description, URDF)
Before this commit: robot red_triangle, 1 links, 0 joints
Links:
- link base_link: mass 0.05 -> 0.000005

Commit message: fixed box weights

File: urdf/blue_box.urdf (robot description, URDF)
Before this commit: robot blue_box, 1 links, 0 joints
Links:
- link base_link: mass 0.005 -> 0.01

File: urdf/red_box.urdf (robot description, URDF)
Before this commit: robot red_box, 1 links, 0 joints
Links:
- link base_link: mass 0.005 -> 0.01

File: urdf/yellow_box.urdf (robot description, URDF)
Before this commit: robot yellow_box, 1 links, 0 joints
Links:
- link base_link: mass 0.000005 -> 0.01
