Commit message: made weights consistent

File: urdf/red_cylinder.urdf (robot description, URDF)
Before this commit: robot red_cylinder, 1 links, 0 joints
Links:
- link base_link: mass 0.005 -> 0.01

File: urdf/yellow_cylinder.urdf (robot description, URDF)
Before this commit: robot yellow_cylinder, 1 links, 0 joints
Links:
- link base_link: mass 0.005 -> 0.01
